Commit message: changed naming in urdf to resolve problems with 'tf_prefix' coming from: https://github.com/ros/robot_state_publisher/pull/139

File: catch/urdf/turtlebot3_burger_cat.gazebo.xacro (robot description, xacro)
@@ -3,8 +3,8 @@
   <xacro:arg name="laser_visual" default="false"/>
   <xacro:arg name="imu_visual"   default="false"/>
-  <gazebo reference="base_link">
+  <gazebo reference="cat/base_link">
     <material>Gazebo/DarkGrey</material>
   </gazebo>
-  <gazebo reference="wheel_left_link">
+  <gazebo reference="cat/wheel_left_link">
     <mu1>0.1</mu1>
     <mu2>0.1</mu2>
@@ -16,5 +16,5 @@
     <material>Gazebo/FlatBlack</material>
   </gazebo>
-  <gazebo reference="wheel_right_link">
+  <gazebo reference="cat/wheel_right_link">
     <mu1>0.1</mu1>
     <mu2>0.1</mu2>
@@ -26,5 +26,5 @@
     <material>Gazebo/FlatBlack</material>
   </gazebo>
-  <gazebo reference="caster_back_link">
+  <gazebo reference="cat/caster_back_link">
     <mu1>0.1</mu1>
     <mu2>0.1</mu2>
@@ -35,5 +35,5 @@
     <material>Gazebo/FlatBlack</material>
   </gazebo>
-  <gazebo reference="imu_link">
+  <gazebo reference="cat/imu_link">
     <sensor type="imu" name="imu">
       <always_on>true</always_on>
@@ -49,5 +49,5 @@
       <odometrySource>world</odometrySource>
       <publishOdomTF>true</publishOdomTF>
-      <robotBaseFrame>base_footprint</robotBaseFrame>
+      <robotBaseFrame>cat/base_footprint</robotBaseFrame>
       <publishWheelTF>false</publishWheelTF>
       <publishTf>true</publishTf>
@@ -55,6 +55,6 @@
       <legacyMode>false</legacyMode>
       <updateRate>30</updateRate>
-      <leftJoint>wheel_left_joint</leftJoint>
-      <rightJoint>wheel_right_joint</rightJoint>
+      <leftJoint>cat/wheel_left_joint</leftJoint>
+      <rightJoint>cat/wheel_right_joint</rightJoint>
       <wheelSeparation>0.160</wheelSeparation>
       <wheelDiameter>0.066</wheelDiameter>
@@ -67,6 +67,6 @@
     <plugin name="imu_plugin" filename="libgazebo_ros_imu.so">
       <alwaysOn>true</alwaysOn>
-      <bodyName>imu_link</bodyName>
-      <frameName>imu_link</frameName>
+      <bodyName>cat/imu_link</bodyName>
+      <frameName>cat/imu_link</frameName>
       <topicName>imu</topicName>
       <serviceName>imu_service</serviceName>
@@ -92,5 +92,5 @@
     </plugin>
   </gazebo>
-  <gazebo reference="base_scan">
+  <gazebo reference="cat/base_scan">
     <material>Gazebo/FlatBlack</material>
     <sensor type="ray" name="lds_lfcd_sensor">
@@ -120,5 +120,5 @@
       <plugin name="gazebo_ros_lds_lfcd_controller" filename="libgazebo_ros_laser.so">
         <topicName>scan</topicName>
-        <frameName>base_scan</frameName>
+        <frameName>cat/base_scan</frameName>
       </plugin>
     </sensor>

File: catch/urdf/turtlebot3_burger_cat.urdf.xacro (robot description, xacro)
@@ -3,11 +3,11 @@
   <xacro:include filename="$(find catch)/urdf/common_properties.xacro"/>
   <xacro:include filename="$(find catch)/urdf/turtlebot3_burger_cat.gazebo.xacro"/>
-  <link name="base_footprint"/>
-  <joint name="base_joint" type="fixed">
-    <parent link="base_footprint"/>
-    <child link="base_link"/>
+  <link name="cat/base_footprint"/>
+  <joint name="cat/base_joint" type="fixed">
+    <parent link="cat/base_footprint"/>
+    <child link="cat/base_link"/>
     <origin xyz="0.0 0.0 0.010" rpy="0 0 0"/>
   </joint>
-  <link name="base_link">
+  <link name="cat/base_link">
     <visual>
       <origin xyz="-0.032 0 0.0" rpy="0 0 0"/>
@@ -31,11 +31,11 @@
     </inertial>
   </link>
-  <joint name="wheel_left_joint" type="continuous">
-    <parent link="base_link"/>
-    <child link="wheel_left_link"/>
+  <joint name="cat/wheel_left_joint" type="continuous">
+    <parent link="cat/base_link"/>
+    <child link="cat/wheel_left_link"/>
     <origin xyz="0.0 0.08 0.023" rpy="-1.57 0 0"/>
     <axis xyz="0 0 1"/>
   </joint>
-  <link name="wheel_left_link">
+  <link name="cat/wheel_left_link">
     <visual>
       <origin xyz="0 0 0" rpy="1.57 0 0"/>
@@ -59,11 +59,11 @@
       </inertial>
   </link>
-  <joint name="wheel_right_joint" type="continuous">
-    <parent link="base_link"/>
-    <child link="wheel_right_link"/>
+  <joint name="cat/wheel_right_joint" type="continuous">
+    <parent link="cat/base_link"/>
+    <child link="cat/wheel_right_link"/>
     <origin xyz="0.0 -0.080 0.023" rpy="-1.57 0 0"/>
     <axis xyz="0 0 1"/>
   </joint>
-  <link name="wheel_right_link">
+  <link name="cat/wheel_right_link">
     <visual>
       <origin xyz="0 0 0" rpy="1.57 0 0"/>
@@ -87,10 +87,10 @@
       </inertial>
   </link>
-  <joint name="caster_back_joint" type="fixed">
-    <parent link="base_link"/>
-    <child link="caster_back_link"/>
+  <joint name="cat/caster_back_joint" type="fixed">
+    <parent link="cat/base_link"/>
+    <child link="cat/caster_back_link"/>
     <origin xyz="-0.081 0 -0.004" rpy="-1.57 0 0"/>
   </joint>
-  <link name="caster_back_link">
+  <link name="cat/caster_back_link">
     <collision>
       <origin xyz="0 0.001 0" rpy="0 0 0"/>
@@ -107,16 +107,16 @@
     </inertial>
   </link>
-  <joint name="imu_joint" type="fixed">
-    <parent link="base_link"/>
-    <child link="imu_link"/>
+  <joint name="cat/imu_joint" type="fixed">
+    <parent link="cat/base_link"/>
+    <child link="cat/imu_link"/>
     <origin xyz="-0.032 0 0.068" rpy="0 0 0"/>
   </joint>
-  <link name="imu_link"/>
-  <joint name="scan_joint" type="fixed">
-    <parent link="base_link"/>
-    <child link="base_scan"/>
+  <link name="cat/imu_link"/>
+  <joint name="cat/scan_joint" type="fixed">
+    <parent link="cat/base_link"/>
+    <child link="cat/base_scan"/>
     <origin xyz="-0.032 0 0.172" rpy="0 0 0"/>
   </joint>
-  <link name="base_scan">
+  <link name="cat/base_scan">
     <visual>
       <origin xyz="0 0 0.0" rpy="0 0 0"/>

File: catch/urdf/turtlebot3_burger_mouse.gazebo.xacro (robot description, xacro)
@@ -3,8 +3,8 @@
   <xacro:arg name="laser_visual" default="false"/>
   <xacro:arg name="imu_visual"   default="false"/>
-  <gazebo reference="base_link">
+  <gazebo reference="mouse/base_link">
     <material>Gazebo/Orange </material>
   </gazebo>
-  <gazebo reference="wheel_left_link">
+  <gazebo reference="mouse/wheel_left_link">
     <mu1>0.1</mu1>
     <mu2>0.1</mu2>
@@ -16,5 +16,5 @@
     <material>Gazebo/FlatBlack</material>
   </gazebo>
-  <gazebo reference="wheel_right_link">
+  <gazebo reference="mouse/wheel_right_link">
     <mu1>0.1</mu1>
     <mu2>0.1</mu2>
@@ -26,5 +26,5 @@
     <material>Gazebo/FlatBlack</material>
   </gazebo>
-  <gazebo reference="caster_back_link">
+  <gazebo reference="mouse/caster_back_link">
     <mu1>0.1</mu1>
     <mu2>0.1</mu2>
@@ -35,5 +35,5 @@
     <material>Gazebo/FlatBlack</material>
   </gazebo>
-  <gazebo reference="imu_link">
+  <gazebo reference="mouse/imu_link">
     <sensor type="imu" name="imu">
       <always_on>true</always_on>
@@ -49,5 +49,5 @@
       <odometrySource>world</odometrySource>
       <publishOdomTF>true</publishOdomTF>
-      <robotBaseFrame>base_footprint</robotBaseFrame>
+      <robotBaseFrame>mouse/base_footprint</robotBaseFrame>
       <publishWheelTF>false</publishWheelTF>
       <publishTf>true</publishTf>
@@ -55,6 +55,6 @@
       <legacyMode>false</legacyMode>
       <updateRate>30</updateRate>
-      <leftJoint>wheel_left_joint</leftJoint>
-      <rightJoint>wheel_right_joint</rightJoint>
+      <leftJoint>mouse/wheel_left_joint</leftJoint>
+      <rightJoint>mouse/wheel_right_joint</rightJoint>
       <wheelSeparation>0.160</wheelSeparation>
       <wheelDiameter>0.066</wheelDiameter>
@@ -67,6 +67,6 @@
     <plugin name="imu_plugin" filename="libgazebo_ros_imu.so">
       <alwaysOn>true</alwaysOn>
-      <bodyName>imu_link</bodyName>
-      <frameName>imu_link</frameName>
+      <bodyName>mouse/imu_link</bodyName>
+      <frameName>mouse/imu_link</frameName>
       <topicName>imu</topicName>
       <serviceName>imu_service</serviceName>
@@ -92,5 +92,5 @@
     </plugin>
   </gazebo>
-  <gazebo reference="base_scan">
+  <gazebo reference="mouse/base_scan">
     <material>Gazebo/FlatBlack</material>
     <sensor type="ray" name="lds_lfcd_sensor">
@@ -120,5 +120,5 @@
       <plugin name="gazebo_ros_lds_lfcd_controller" filename="libgazebo_ros_laser.so">
         <topicName>scan</topicName>
-        <frameName>base_scan</frameName>
+        <frameName>mouse/base_scan</frameName>
       </plugin>
     </sensor>

File: catch/urdf/turtlebot3_burger_mouse.urdf.xacro (robot description, xacro)
@@ -3,11 +3,11 @@
   <xacro:include filename="$(find catch)/urdf/common_properties.xacro"/>
   <xacro:include filename="$(find catch)/urdf/turtlebot3_burger_mouse.gazebo.xacro"/>
-  <link name="base_footprint"/>
-  <joint name="base_joint" type="fixed">
-    <parent link="base_footprint"/>
-    <child link="base_link"/>
+  <link name="mouse/base_footprint"/>
+  <joint name="mouse/base_joint" type="fixed">
+    <parent link="mouse/base_footprint"/>
+    <child link="mouse/base_link"/>
     <origin xyz="0.0 0.0 0.010" rpy="0 0 0"/>
   </joint>
-  <link name="base_link">
+  <link name="mouse/base_link">
     <visual>
       <origin xyz="-0.032 0 0.0" rpy="0 0 0"/>
@@ -31,11 +31,11 @@
     </inertial>
   </link>
-  <joint name="wheel_left_joint" type="continuous">
-    <parent link="base_link"/>
-    <child link="wheel_left_link"/>
+  <joint name="mouse/wheel_left_joint" type="continuous">
+    <parent link="mouse/base_link"/>
+    <child link="mouse/wheel_left_link"/>
     <origin xyz="0.0 0.08 0.023" rpy="-1.57 0 0"/>
     <axis xyz="0 0 1"/>
   </joint>
-  <link name="wheel_left_link">
+  <link name="mouse/wheel_left_link">
     <visual>
       <origin xyz="0 0 0" rpy="1.57 0 0"/>
@@ -59,11 +59,11 @@
       </inertial>
   </link>
-  <joint name="wheel_right_joint" type="continuous">
-    <parent link="base_link"/>
-    <child link="wheel_right_link"/>
+  <joint name="mouse/wheel_right_joint" type="continuous">
+    <parent link="mouse/base_link"/>
+    <child link="mouse/wheel_right_link"/>
     <origin xyz="0.0 -0.080 0.023" rpy="-1.57 0 0"/>
     <axis xyz="0 0 1"/>
   </joint>
-  <link name="wheel_right_link">
+  <link name="mouse/wheel_right_link">
     <visual>
       <origin xyz="0 0 0" rpy="1.57 0 0"/>
@@ -87,10 +87,10 @@
       </inertial>
   </link>
-  <joint name="caster_back_joint" type="fixed">
-    <parent link="base_link"/>
-    <child link="caster_back_link"/>
+  <joint name="mouse/caster_back_joint" type="fixed">
+    <parent link="mouse/base_link"/>
+    <child link="mouse/caster_back_link"/>
     <origin xyz="-0.081 0 -0.004" rpy="-1.57 0 0"/>
   </joint>
-  <link name="caster_back_link">
+  <link name="mouse/caster_back_link">
     <collision>
       <origin xyz="0 0.001 0" rpy="0 0 0"/>
@@ -107,16 +107,16 @@
     </inertial>
   </link>
-  <joint name="imu_joint" type="fixed">
-    <parent link="base_link"/>
-    <child link="imu_link"/>
+  <joint name="mouse/imu_joint" type="fixed">
+    <parent link="mouse/base_link"/>
+    <child link="mouse/imu_link"/>
     <origin xyz="-0.032 0 0.068" rpy="0 0 0"/>
   </joint>
-  <link name="imu_link"/>
-  <joint name="scan_joint" type="fixed">
-    <parent link="base_link"/>
-    <child link="base_scan"/>
+  <link name="mouse/imu_link"/>
+  <joint name="mouse/scan_joint" type="fixed">
+    <parent link="mouse/base_link"/>
+    <child link="mouse/base_scan"/>
     <origin xyz="-0.032 0 0.172" rpy="0 0 0"/>
   </joint>
-  <link name="base_scan">
+  <link name="mouse/base_scan">
     <visual>
       <origin xyz="0 0 0.0" rpy="0 0 0"/>

File: heist/urdf/turtlebot3_burger_green.gazebo.xacro (robot description, xacro)
@@ -3,8 +3,8 @@
   <xacro:arg name="laser_visual" default="false"/>
   <xacro:arg name="imu_visual"   default="false"/>
-  <gazebo reference="base_link">
+  <gazebo reference="evader/base_link">
     <material>Gazebo/Green </material>
   </gazebo>
-  <gazebo reference="wheel_left_link">
+  <gazebo reference="evader/wheel_left_link">
     <mu1>0.1</mu1>
     <mu2>0.1</mu2>
@@ -16,5 +16,5 @@
     <material>Gazebo/FlatBlack</material>
   </gazebo>
-  <gazebo reference="wheel_right_link">
+  <gazebo reference="evader/wheel_right_link">
     <mu1>0.1</mu1>
     <mu2>0.1</mu2>
@@ -26,5 +26,5 @@
     <material>Gazebo/FlatBlack</material>
   </gazebo>
-  <gazebo reference="caster_back_link">
+  <gazebo reference="evader/caster_back_link">
     <mu1>0.1</mu1>
     <mu2>0.1</mu2>
@@ -35,5 +35,5 @@
     <material>Gazebo/FlatBlack</material>
   </gazebo>
-  <gazebo reference="imu_link">
+  <gazebo reference="evader/imu_link">
     <sensor type="imu" name="imu">
       <always_on>true</always_on>
@@ -49,5 +49,5 @@
       <odometrySource>world</odometrySource>
       <publishOdomTF>true</publishOdomTF>
-      <robotBaseFrame>base_footprint</robotBaseFrame>
+      <robotBaseFrame>evader/base_footprint</robotBaseFrame>
       <publishWheelTF>false</publishWheelTF>
       <publishTf>true</publishTf>
@@ -55,6 +55,6 @@
       <legacyMode>false</legacyMode>
       <updateRate>30</updateRate>
-      <leftJoint>wheel_left_joint</leftJoint>
-      <rightJoint>wheel_right_joint</rightJoint>
+      <leftJoint>evader/wheel_left_joint</leftJoint>
+      <rightJoint>evader/wheel_right_joint</rightJoint>
       <wheelSeparation>0.160</wheelSeparation>
       <wheelDiameter>0.066</wheelDiameter>
@@ -67,6 +67,6 @@
     <plugin name="imu_plugin" filename="libgazebo_ros_imu.so">
       <alwaysOn>true</alwaysOn>
-      <bodyName>imu_link</bodyName>
-      <frameName>imu_link</frameName>
+      <bodyName>evader/imu_link</bodyName>
+      <frameName>evader/imu_link</frameName>
       <topicName>imu</topicName>
       <serviceName>imu_service</serviceName>
@@ -92,5 +92,5 @@
     </plugin>
   </gazebo>
-  <gazebo reference="base_scan">
+  <gazebo reference="evader/base_scan">
     <material>Gazebo/FlatBlack</material>
     <sensor type="ray" name="lds_lfcd_sensor">
@@ -120,5 +120,5 @@
       <plugin name="gazebo_ros_lds_lfcd_controller" filename="libgazebo_ros_laser.so">
         <topicName>scan</topicName>
-        <frameName>base_scan</frameName>
+        <frameName>evader/base_scan</frameName>
       </plugin>
     </sensor>

File: heist/urdf/turtlebot3_burger_green.urdf.xacro (robot description, xacro)
@@ -3,11 +3,11 @@
   <xacro:include filename="$(find heist)/urdf/common_properties.xacro"/>
   <xacro:include filename="$(find heist)/urdf/turtlebot3_burger_green.gazebo.xacro"/>
-  <link name="base_footprint"/>
-  <joint name="base_joint" type="fixed">
-    <parent link="base_footprint"/>
-    <child link="base_link"/>
+  <link name="evader/base_footprint"/>
+  <joint name="evader/base_joint" type="fixed">
+    <parent link="evader/base_footprint"/>
+    <child link="evader/base_link"/>
     <origin xyz="0.0 0.0 0.010" rpy="0 0 0"/>
   </joint>
-  <link name="base_link">
+  <link name="evader/base_link">
     <visual>
       <origin xyz="-0.032 0 0.0" rpy="0 0 0"/>
@@ -31,11 +31,11 @@
     </inertial>
   </link>
-  <joint name="wheel_left_joint" type="continuous">
-    <parent link="base_link"/>
-    <child link="wheel_left_link"/>
+  <joint name="evader/wheel_left_joint" type="continuous">
+    <parent link="evader/base_link"/>
+    <child link="evader/wheel_left_link"/>
     <origin xyz="0.0 0.08 0.023" rpy="-1.57 0 0"/>
     <axis xyz="0 0 1"/>
   </joint>
-  <link name="wheel_left_link">
+  <link name="evader/wheel_left_link">
     <visual>
       <origin xyz="0 0 0" rpy="1.57 0 0"/>
@@ -59,11 +59,11 @@
       </inertial>
   </link>
-  <joint name="wheel_right_joint" type="continuous">
-    <parent link="base_link"/>
-    <child link="wheel_right_link"/>
+  <joint name="evader/wheel_right_joint" type="continuous">
+    <parent link="evader/base_link"/>
+    <child link="evader/wheel_right_link"/>
     <origin xyz="0.0 -0.080 0.023" rpy="-1.57 0 0"/>
     <axis xyz="0 0 1"/>
   </joint>
-  <link name="wheel_right_link">
+  <link name="evader/wheel_right_link">
     <visual>
       <origin xyz="0 0 0" rpy="1.57 0 0"/>
@@ -87,10 +87,10 @@
       </inertial>
   </link>
-  <joint name="caster_back_joint" type="fixed">
-    <parent link="base_link"/>
-    <child link="caster_back_link"/>
+  <joint name="evader/caster_back_joint" type="fixed">
+    <parent link="evader/base_link"/>
+    <child link="evader/caster_back_link"/>
     <origin xyz="-0.081 0 -0.004" rpy="-1.57 0 0"/>
   </joint>
-  <link name="caster_back_link">
+  <link name="evader/caster_back_link">
     <collision>
       <origin xyz="0 0.001 0" rpy="0 0 0"/>
@@ -107,16 +107,16 @@
     </inertial>
   </link>
-  <joint name="imu_joint" type="fixed">
-    <parent link="base_link"/>
-    <child link="imu_link"/>
+  <joint name="evader/imu_joint" type="fixed">
+    <parent link="evader/base_link"/>
+    <child link="evader/imu_link"/>
     <origin xyz="-0.032 0 0.068" rpy="0 0 0"/>
   </joint>
-  <link name="imu_link"/>
-  <joint name="scan_joint" type="fixed">
-    <parent link="base_link"/>
-    <child link="base_scan"/>
+  <link name="evader/imu_link"/>
+  <joint name="evader/scan_joint" type="fixed">
+    <parent link="evader/base_link"/>
+    <child link="evader/base_scan"/>
     <origin xyz="-0.032 0 0.172" rpy="0 0 0"/>
   </joint>
-  <link name="base_scan">
+  <link name="evader/base_scan">
     <visual>
       <origin xyz="0 0 0.0" rpy="0 0 0"/>

File: heist/urdf/turtlebot3_burger_red.gazebo.xacro (robot description, xacro)
@@ -3,8 +3,8 @@
   <xacro:arg name="laser_visual" default="false"/>
   <xacro:arg name="imu_visual"   default="false"/>
-  <gazebo reference="base_link">
+  <gazebo reference="guard/base_link">
     <material>Gazebo/Red</material>
   </gazebo>
-  <gazebo reference="wheel_left_link">
+  <gazebo reference="guard/wheel_left_link">
     <mu1>0.1</mu1>
     <mu2>0.1</mu2>
@@ -16,5 +16,5 @@
     <material>Gazebo/FlatBlack</material>
   </gazebo>
-  <gazebo reference="wheel_right_link">
+  <gazebo reference="guard/wheel_right_link">
     <mu1>0.1</mu1>
     <mu2>0.1</mu2>
@@ -26,5 +26,5 @@
     <material>Gazebo/FlatBlack</material>
   </gazebo>
-  <gazebo reference="caster_back_link">
+  <gazebo reference="guard/caster_back_link">
     <mu1>0.1</mu1>
     <mu2>0.1</mu2>
@@ -35,5 +35,5 @@
     <material>Gazebo/FlatBlack</material>
   </gazebo>
-  <gazebo reference="imu_link">
+  <gazebo reference="guard/imu_link">
     <sensor type="imu" name="imu">
       <always_on>true</always_on>
@@ -49,5 +49,5 @@
       <odometrySource>world</odometrySource>
       <publishOdomTF>true</publishOdomTF>
-      <robotBaseFrame>base_footprint</robotBaseFrame>
+      <robotBaseFrame>guard/base_footprint</robotBaseFrame>
       <publishWheelTF>false</publishWheelTF>
       <publishTf>true</publishTf>
@@ -55,6 +55,6 @@
       <legacyMode>false</legacyMode>
       <updateRate>30</updateRate>
-      <leftJoint>wheel_left_joint</leftJoint>
-      <rightJoint>wheel_right_joint</rightJoint>
+      <leftJoint>guard/wheel_left_joint</leftJoint>
+      <rightJoint>guard/wheel_right_joint</rightJoint>
       <wheelSeparation>0.160</wheelSeparation>
       <wheelDiameter>0.066</wheelDiameter>
@@ -67,6 +67,6 @@
     <plugin name="imu_plugin" filename="libgazebo_ros_imu.so">
       <alwaysOn>true</alwaysOn>
-      <bodyName>imu_link</bodyName>
-      <frameName>imu_link</frameName>
+      <bodyName>guard/imu_link</bodyName>
+      <frameName>guard/imu_link</frameName>
       <topicName>imu</topicName>
       <serviceName>imu_service</serviceName>
@@ -92,5 +92,5 @@
     </plugin>
   </gazebo>
-  <gazebo reference="base_scan">
+  <gazebo reference="guard/base_scan">
     <material>Gazebo/FlatBlack</material>
     <sensor type="ray" name="lds_lfcd_sensor">
@@ -120,5 +120,5 @@
       <plugin name="gazebo_ros_lds_lfcd_controller" filename="libgazebo_ros_laser.so">
         <topicName>scan</topicName>
-        <frameName>base_scan</frameName>
+        <frameName>guard/base_scan</frameName>
       </plugin>
     </sensor>

File: heist/urdf/turtlebot3_burger_red.urdf.xacro (robot description, xacro)
@@ -3,11 +3,11 @@
   <xacro:include filename="$(find heist)/urdf/common_properties.xacro"/>
   <xacro:include filename="$(find heist)/urdf/turtlebot3_burger_red.gazebo.xacro"/>
-  <link name="base_footprint"/>
-  <joint name="base_joint" type="fixed">
-    <parent link="base_footprint"/>
-    <child link="base_link"/>
+  <link name="guard/base_footprint"/>
+  <joint name="guard/base_joint" type="fixed">
+    <parent link="guard/base_footprint"/>
+    <child link="guard/base_link"/>
     <origin xyz="0.0 0.0 0.010" rpy="0 0 0"/>
   </joint>
-  <link name="base_link">
+  <link name="guard/base_link">
     <visual>
       <origin xyz="-0.032 0 0.0" rpy="0 0 0"/>
@@ -31,11 +31,11 @@
     </inertial>
   </link>
-  <joint name="wheel_left_joint" type="continuous">
-    <parent link="base_link"/>
-    <child link="wheel_left_link"/>
+  <joint name="guard/wheel_left_joint" type="continuous">
+    <parent link="guard/base_link"/>
+    <child link="guard/wheel_left_link"/>
     <origin xyz="0.0 0.08 0.023" rpy="-1.57 0 0"/>
     <axis xyz="0 0 1"/>
   </joint>
-  <link name="wheel_left_link">
+  <link name="guard/wheel_left_link">
     <visual>
       <origin xyz="0 0 0" rpy="1.57 0 0"/>
@@ -59,11 +59,11 @@
       </inertial>
   </link>
-  <joint name="wheel_right_joint" type="continuous">
-    <parent link="base_link"/>
-    <child link="wheel_right_link"/>
+  <joint name="guard/wheel_right_joint" type="continuous">
+    <parent link="guard/base_link"/>
+    <child link="guard/wheel_right_link"/>
     <origin xyz="0.0 -0.080 0.023" rpy="-1.57 0 0"/>
     <axis xyz="0 0 1"/>
   </joint>
-  <link name="wheel_right_link">
+  <link name="guard/wheel_right_link">
     <visual>
       <origin xyz="0 0 0" rpy="1.57 0 0"/>
@@ -87,10 +87,10 @@
       </inertial>
   </link>
-  <joint name="caster_back_joint" type="fixed">
-    <parent link="base_link"/>
-    <child link="caster_back_link"/>
+  <joint name="guard/caster_back_joint" type="fixed">
+    <parent link="guard/base_link"/>
+    <child link="guard/caster_back_link"/>
     <origin xyz="-0.081 0 -0.004" rpy="-1.57 0 0"/>
   </joint>
-  <link name="caster_back_link">
+  <link name="guard/caster_back_link">
     <collision>
       <origin xyz="0 0.001 0" rpy="0 0 0"/>
@@ -107,16 +107,16 @@
     </inertial>
   </link>
-  <joint name="imu_joint" type="fixed">
-    <parent link="base_link"/>
-    <child link="imu_link"/>
+  <joint name="guard/imu_joint" type="fixed">
+    <parent link="guard/base_link"/>
+    <child link="guard/imu_link"/>
     <origin xyz="-0.032 0 0.068" rpy="0 0 0"/>
   </joint>
-  <link name="imu_link"/>
-  <joint name="scan_joint" type="fixed">
-    <parent link="base_link"/>
-    <child link="base_scan"/>
+  <link name="guard/imu_link"/>
+  <joint name="guard/scan_joint" type="fixed">
+    <parent link="guard/base_link"/>
+    <child link="guard/base_scan"/>
     <origin xyz="-0.032 0 0.172" rpy="0 0 0"/>
   </joint>
-  <link name="base_scan">
+  <link name="guard/base_scan">
     <visual>
       <origin xyz="0 0 0.0" rpy="0 0 0"/>
